Commit message: Fix measurements for the new car

File: src/auto/urdf/auto.urdf (robot description, URDF)
Before this commit: robot tx2-auto-3, 14 links, 13 joints
Joints:
- joint f_axle_joint: origin xyz=0.16 0 0.0525 rpy=0 0 0 -> xyz=0.1635 0 0.0525 rpy=0 0 0
- joint imu_link_joint: origin xyz=0.025 0 0.095 -> xyz=0.1265 0 0.005
- joint lf_wheel_joint: origin xyz=0.16 0.115 0.0525 rpy=0 0 0 -> xyz=0.1635 0.125 0.0525 rpy=0 0 0
- joint lidar_base_joint: origin xyz=0.025 0 0.105 -> xyz=0.1265 0 0.015
- joint lr_wheel_joint: origin xyz=-0.16 0.115 0.0525 rpy=0 0 0 -> xyz=-0.1635 0.125 0.0525 rpy=0 0 0
- joint r_axle_joint: origin xyz=-0.16 0 0.0525 rpy=0 0 0 -> xyz=-0.1635 0 0.0525 rpy=0 0 0
- joint rf_wheel_joint: origin xyz=0.16 -0.115 0.0525 rpy=0 0 0 -> xyz=0.1635 -0.125 0.0525 rpy=0 0 0
- joint rr_wheel_joint: origin xyz=-0.16 -0.115 0.0525 rpy=0 0 0 -> xyz=-0.1635 -0.125 0.0525 rpy=0 0 0
